File: breakout-boards/eeprom/eeprom.sch (KiCad schematic (older format))
At the start: 8 parts, among them J1 BREAKOUT, U1 AP2127N-3.3, U2 M95256-WMN6P

Commit message: (#14) redo stm32 and eeprom board to only include 0603 and 0805 components
Parts:
- C1, C3: footprint Capacitor_SMD:C_0402_1005Metric -> Capacitor_SMD:C_0603_1608Metric
- C2, C5: footprint Capacitor_SMD:C_0201_0603Metric -> Capacitor_SMD:C_0603_1608Metric
- C4: footprint Capacitor_SMD:C_0805_2012Metric -> Capacitor_SMD:C_0603_1608Metric
Changed lines of the file:
@@
 F 0 "C5" H 5742 3496 50  0000 L CNN
 F 1 "C_100nF" H 5742 3405 50  0000 L CNN
-F 2 "Capacitor_SMD:C_0201_0603Metric" H 5825 3450 50  0001 C CNN
+F 2 "Capacitor_SMD:C_0603_1608Metric" H 5825 3450 50  0001 C CNN
 F 3 "" H 5825 3450 50  0001 C CNN
 	1    5650 3450
@@
 F 0 "C4" H 5292 3496 50  0000 L CNN
 F 1 "C_10uF" H 5292 3405 50  0000 L CNN
-F 2 "Capacitor_SMD:C_0805_2012Metric" H 5200 3450 50  0001 C CNN
+F 2 "Capacitor_SMD:C_0603_1608Metric" H 5200 3450 50  0001 C CNN
 F 3 "" H 5200 3450 50  0001 C CNN
 	1    5200 3450
@@
 F 0 "C2" H 2392 3546 50  0000 L CNN
 F 1 "C_100nF" H 2392 3455 50  0000 L CNN
-F 2 "Capacitor_SMD:C_0201_0603Metric" H 2475 3500 50  0001 C CNN
+F 2 "Capacitor_SMD:C_0603_1608Metric" H 2475 3500 50  0001 C CNN
 F 3 "" H 2475 3500 50  0001 C CNN
 	1    2300 3500
@@
 F 0 "C1" H 1992 3546 50  0000 L CNN
 F 1 "C_1uF" H 1992 3455 50  0000 L CNN
-F 2 "Capacitor_SMD:C_0402_1005Metric" H 2175 3550 50  0001 C CNN
+F 2 "Capacitor_SMD:C_0603_1608Metric" H 2175 3550 50  0001 C CNN
 F 3 "" H 2050 3500 50  0001 C CNN
 	1    1900 3500
@@
 F 0 "C3" H 3542 3546 50  0000 L CNN
 F 1 "C_4.7uF" H 3542 3455 50  0000 L CNN
-F 2 "Capacitor_SMD:C_0402_1005Metric" H 3725 3550 50  0001 C CNN
+F 2 "Capacitor_SMD:C_0603_1608Metric" H 3725 3550 50  0001 C CNN
 F 3 "" H 3600 3500 50  0001 C CNN
 	1    3450 3500
